Commit message: Add PGI Gazebo simulation and gripper control

File: urdf/pgi_140_80_macro.xacro (robot description, xacro)
@@ -14,9 +14,39 @@
     manufacturing geometry or as a real-robot payload/TCP calibration.
   -->
-  <xacro:macro name="pgi_140_80" params="parent prefix camera_mount_xyz camera_mount_rpy">
+  <!-- Uniform-box inertia helper for explicitly provisional Gazebo masses.
+       These values make the temporary primitives numerically well-formed;
+       they are not manufacturer or payload-calibration data. -->
+  <xacro:macro name="pgi_provisional_box_inertial"
+               params="mass size_x size_y size_z origin_xyz">
+    <inertial>
+      <origin xyz="${origin_xyz}" rpy="0 0 0"/>
+      <mass value="${mass}"/>
+      <inertia
+        ixx="${mass * (size_y * size_y + size_z * size_z) / 12.0}"
+        ixy="0" ixz="0"
+        iyy="${mass * (size_x * size_x + size_z * size_z) / 12.0}"
+        iyz="0"
+        izz="${mass * (size_x * size_x + size_y * size_y) / 12.0}"/>
+    </inertial>
+  </xacro:macro>
+  <xacro:macro name="pgi_140_80"
+               params="parent prefix camera_mount_xyz camera_mount_rpy use_gz_ros2_control:=false">
+    <!-- The nominal and commandable travel remains 0.040 m per jaw. DART can
+         latch a position-controlled prismatic joint after it is held exactly
+         against a hard stop, so the Gazebo-only hard stop has a 0.5 mm
+         numerical guard band. ros2_control command-limit enforcement keeps
+         this guard band unreachable through GripperCommand. -->
+    <xacro:property name="pgi_physics_upper_limit" value="0.040"/>
+    <xacro:if value="${use_gz_ros2_control}">
+      <xacro:property name="pgi_physics_upper_limit" value="0.0405"/>
+    </xacro:if>
     <!-- Placeholder camera interposer. Its final material, mass, and geometry
-         depend on the project adapter design and are intentionally not given
-         an inertial block. The joint origin is the UR tool0/F1 interface. -->
+         depend on the project adapter design. The 0.10 kg uniform-box inertia
+         is a provisional Gazebo stability value, not a verified adapter mass.
+         The joint origin is the UR tool0/F1 interface. -->
     <link name="${prefix}pgi_camera_interposer">
+      <xacro:pgi_provisional_box_inertial
+        mass="${0.10}" size_x="${0.085}" size_y="${0.085}"
+        size_z="${0.010}" origin_xyz="0 0 0.005"/>
       <visual name="provisional_interposer_visual">
         <origin xyz="0 0 0.005" rpy="0 0 0"/>
@@ -39,4 +69,9 @@
          50 mm pitch circle. Bolt and pilot holes are omitted from collision. -->
     <link name="${prefix}pgi_mount">
+      <!-- 0.08 kg is provisional. The box inertia encloses the temporary F1
+           cylinder and must be replaced with CAD-derived data. -->
+      <xacro:pgi_provisional_box_inertial
+        mass="${0.08}" size_x="${0.063}" size_y="${0.063}"
+        size_z="${0.0065}" origin_xyz="0 0 0.00325"/>
       <visual name="provisional_f1_visual">
         <origin xyz="0 0 0.00325" rpy="0 0 0"/>
@@ -83,4 +118,9 @@
          faces meet at body X=0. Positive q opens each jaw by 40 mm. -->
     <link name="${prefix}pgi_left_finger">
+      <!-- Exact J1 mass is unavailable; 0.05 kg is a provisional value used
+           only to keep the moving Gazebo link dynamically valid. -->
+      <xacro:pgi_provisional_box_inertial
+        mass="${0.05}" size_x="${0.015}" size_y="${0.020}"
+        size_z="${0.050}" origin_xyz="0.0075 0 0.025"/>
       <visual name="provisional_j1_left_visual">
         <origin xyz="0.0075 0 0.025" rpy="0 0 0"/>
@@ -98,7 +138,12 @@
       <child link="${prefix}pgi_left_finger"/>
       <axis xyz="1 0 0"/>
-      <limit lower="0.0" upper="0.040" effort="140.0" velocity="0.0364"/>
+      <limit lower="0.0" upper="${pgi_physics_upper_limit}" effort="140.0" velocity="0.0364"/>
+      <!-- Provisional viscous damping for stable position control in Gazebo. -->
+      <dynamics damping="2.0" friction="0.0"/>
     </joint>
     <link name="${prefix}pgi_right_finger">
+      <xacro:pgi_provisional_box_inertial
+        mass="${0.05}" size_x="${0.015}" size_y="${0.020}"
+        size_z="${0.050}" origin_xyz="-0.0075 0 0.025"/>
       <visual name="provisional_j1_right_visual">
         <origin xyz="-0.0075 0 0.025" rpy="0 0 0"/>
@@ -116,5 +161,6 @@
       <child link="${prefix}pgi_right_finger"/>
       <axis xyz="-1 0 0"/>
-      <limit lower="0.0" upper="0.040" effort="140.0" velocity="0.0364"/>
+      <limit lower="0.0" upper="${pgi_physics_upper_limit}" effort="140.0" velocity="0.0364"/>
+      <dynamics damping="2.0" friction="0.0"/>
       <mimic joint="${prefix}pgi_left_finger_joint" multiplier="1.0" offset="0.0"/>
     </joint>
@@ -129,6 +175,10 @@
     <!-- The camera transform is an opt-in simulation parameter and does not
          modify config/ur10e_real/d435i_mount_calibration.json. The mount and
-         camera boxes are placeholders with no asserted mass properties. -->
+         camera boxes are placeholders. Their masses below are explicitly
+         provisional Gazebo values, not asserted camera/adapter properties. -->
     <link name="${prefix}d435i_mount">
+      <xacro:pgi_provisional_box_inertial
+        mass="${0.05}" size_x="${0.095}" size_y="${0.030}"
+        size_z="${0.015}" origin_xyz="0 0 0.0075"/>
       <visual name="provisional_d435i_mount_visual">
         <origin xyz="0 0 0.0075" rpy="0 0 0"/>
@@ -147,4 +197,7 @@
     </joint>
     <link name="${prefix}d435i_link">
+      <xacro:pgi_provisional_box_inertial
+        mass="${0.10}" size_x="${0.090}" size_y="${0.025}"
+        size_z="${0.025}" origin_xyz="0 0 0.0125"/>
       <visual name="provisional_d435i_body_visual">
         <origin xyz="0 0 0.0125" rpy="0 0 0"/>
@@ -176,4 +229,53 @@
       <child link="${prefix}d435i_depth_optical_frame"/>
     </joint>
+    <!-- Keep the fixed attachment links as distinct Gazebo entities so their
+         names and frames remain inspectable. Massless logical/optical frames
+         are still published by robot_state_publisher. -->
+    <gazebo reference="${prefix}tool0-pgi_camera_interposer">
+      <preserveFixedJoint>true</preserveFixedJoint>
+    </gazebo>
+    <gazebo reference="${prefix}pgi_camera_interposer-pgi_mount">
+      <preserveFixedJoint>true</preserveFixedJoint>
+    </gazebo>
+    <gazebo reference="${prefix}pgi_mount-pgi_body">
+      <preserveFixedJoint>true</preserveFixedJoint>
+    </gazebo>
+    <gazebo reference="${prefix}pgi_camera_interposer-d435i_mount">
+      <preserveFixedJoint>true</preserveFixedJoint>
+    </gazebo>
+    <gazebo reference="${prefix}d435i_mount-d435i_link">
+      <preserveFixedJoint>true</preserveFixedJoint>
+    </gazebo>
+    <!-- Logical grasp/optical frames intentionally have no mass. They remain
+         ROS TF frames, but are allowed to lump into their fixed parents during
+         URDF-to-SDF conversion instead of inventing fake inertial data. -->
+    <!-- Gazebo control is a separate opt-in from visualizing the PGI model.
+         Only the left/master jaw exposes a command interface. The right jaw
+         is a passive mimic and exposes state only, as required by ros2_control. -->
+    <xacro:if value="${use_gz_ros2_control}">
+      <ros2_control name="${prefix}pgi_140_80_sim_system" type="system">
+        <hardware>
+          <plugin>gz_ros2_control/GazeboSimSystem</plugin>
+        </hardware>
+        <joint name="${prefix}pgi_left_finger_joint">
+          <command_interface name="position">
+            <param name="min">0.0</param>
+            <param name="max">0.040</param>
+          </command_interface>
+          <state_interface name="position">
+            <param name="initial_value">0.040</param>
+          </state_interface>
+          <state_interface name="velocity"/>
+          <state_interface name="effort"/>
+        </joint>
+        <joint name="${prefix}pgi_right_finger_joint">
+          <state_interface name="position">
+            <param name="initial_value">0.040</param>
+          </state_interface>
+          <state_interface name="velocity"/>
+          <state_interface name="effort"/>
+        </joint>
+      </ros2_control>
+    </xacro:if>
   </xacro:macro>
 </robot>

File: urdf/ur_gz_feeding_markers.urdf.xacro (robot description, xacro)
@@ -31,4 +31,5 @@
        real D435i calibration or the default feeding model. -->
   <xacro:arg name="use_pgi_gripper" default="false" />
+  <xacro:arg name="use_pgi_sim_control" default="false" />
   <xacro:arg name="camera_mount_xyz" default="0 -0.065 0.020" />
   <xacro:arg name="camera_mount_rpy" default="0 0 0" />
@@ -81,4 +82,5 @@
       camera_mount_xyz="$(arg camera_mount_xyz)"
       camera_mount_rpy="$(arg camera_mount_rpy)"
+      use_gz_ros2_control="$(arg use_pgi_sim_control)"
     />
   </xacro:if>

Commit message: Add PGI RGB-D cup perception and tapered grasp model

File: urdf/pgi_140_80_macro.xacro (robot description, xacro)
@@ -126,5 +126,7 @@
         <origin xyz="0.0075 0 0.025" rpy="0 0 0"/>
         <geometry><box size="0.015 0.020 0.050"/></geometry>
-        <material name="pgi_finger_blue"><color rgba="0.10 0.32 0.62 1"/></material>
+        <!-- Neutral provisional fingertip color prevents the basic blue-cup
+             observer from mistaking robot self-geometry for the target. -->
+        <material name="pgi_finger_dark"><color rgba="0.18 0.20 0.23 1"/></material>
       </visual>
       <collision name="simplified_j1_left_collision">
@@ -149,5 +151,5 @@
         <origin xyz="-0.0075 0 0.025" rpy="0 0 0"/>
         <geometry><box size="0.015 0.020 0.050"/></geometry>
-        <material name="pgi_finger_blue_right"><color rgba="0.10 0.32 0.62 1"/></material>
+        <material name="pgi_finger_dark_right"><color rgba="0.18 0.20 0.23 1"/></material>
       </visual>
       <collision name="simplified_j1_right_collision">
@@ -179,14 +181,14 @@
     <link name="${prefix}d435i_mount">
       <xacro:pgi_provisional_box_inertial
-        mass="${0.05}" size_x="${0.095}" size_y="${0.030}"
+        mass="${0.05}" size_x="${0.030}" size_y="${0.095}"
         size_z="${0.015}" origin_xyz="0 0 0.0075"/>
       <visual name="provisional_d435i_mount_visual">
         <origin xyz="0 0 0.0075" rpy="0 0 0"/>
-        <geometry><box size="0.095 0.030 0.015"/></geometry>
+        <geometry><box size="0.030 0.095 0.015"/></geometry>
         <material name="d435i_mount_gray"><color rgba="0.35 0.37 0.40 1"/></material>
       </visual>
       <collision name="provisional_d435i_mount_collision">
         <origin xyz="0 0 0.0075" rpy="0 0 0"/>
-        <geometry><box size="0.095 0.030 0.015"/></geometry>
+        <geometry><box size="0.030 0.095 0.015"/></geometry>
       </collision>
     </link>
@@ -198,14 +200,14 @@
     <link name="${prefix}d435i_link">
       <xacro:pgi_provisional_box_inertial
-        mass="${0.10}" size_x="${0.090}" size_y="${0.025}"
+        mass="${0.10}" size_x="${0.025}" size_y="${0.090}"
         size_z="${0.025}" origin_xyz="0 0 0.0125"/>
       <visual name="provisional_d435i_body_visual">
         <origin xyz="0 0 0.0125" rpy="0 0 0"/>
-        <geometry><box size="0.090 0.025 0.025"/></geometry>
+        <geometry><box size="0.025 0.090 0.025"/></geometry>
         <material name="d435i_body_black"><color rgba="0.05 0.05 0.06 1"/></material>
       </visual>
       <collision name="provisional_d435i_body_collision">
         <origin xyz="0 0 0.0125" rpy="0 0 0"/>
-        <geometry><box size="0.090 0.025 0.025"/></geometry>
+        <geometry><box size="0.025 0.090 0.025"/></geometry>
       </collision>
     </link>
@@ -229,4 +231,34 @@
       <child link="${prefix}d435i_depth_optical_frame"/>
     </joint>
+    <!-- Ideal registered RGB-D source for the simulation-only PGI camera.
+         The topic/message contract mirrors the earlier wrist RGB-D
+         simulation so perception can later switch to aligned real D435i
+         topics without changing its output contract or the planning layer. -->
+    <gazebo reference="${prefix}d435i_link">
+      <sensor name="pgi_d435i" type="rgbd_camera">
+        <!-- Place the rendered sensor at the same provisional baseline as
+             d435i_depth_optical_frame. Gazebo supplies the optical-axis
+             convention internally, so only the link-frame translation is
+             applied here. -->
+        <pose>-0.015 0 0.0125 0 0 0</pose>
+        <always_on>1</always_on>
+        <update_rate>15</update_rate>
+        <visualize>false</visualize>
+        <topic>/pgi_d435i</topic>
+        <camera>
+          <horizontal_fov>1.600</horizontal_fov>
+          <image>
+            <width>640</width>
+            <height>480</height>
+            <format>R8G8B8</format>
+          </image>
+          <clip>
+            <near>0.05</near>
+            <far>3.0</far>
+          </clip>
+          <optical_frame_id>${prefix}d435i_depth_optical_frame</optical_frame_id>
+        </camera>
+      </sensor>
+    </gazebo>
     <!-- Keep the fixed attachment links as distinct Gazebo entities so their
          names and frames remain inspectable. Massless logical/optical frames

File: urdf/ur_gz_feeding_markers.urdf.xacro (robot description, xacro)
@@ -32,6 +32,9 @@
   <xacro:arg name="use_pgi_gripper" default="false" />
   <xacro:arg name="use_pgi_sim_control" default="false" />
-  <xacro:arg name="camera_mount_xyz" default="0 -0.065 0.020" />
-  <xacro:arg name="camera_mount_rpy" default="0 0 0" />
+  <xacro:arg name="camera_mount_xyz" default="0 0.085 0.030" />
+  <!-- The provisional side-front mount rotates the camera optical +Z onto
+       tool0 +Z. With the flange-down constraint, it looks toward the ground
+       and grasp region without tilting the flange. -->
+  <xacro:arg name="camera_mount_rpy" default="0 -1.57079632679 0" />
   <!-- Initial camera-ready pose: tool0 +Z points along world -Z (down). -->
   <xacro:property name="feeding_initial_positions" value="${dict(shoulder_pan_joint=-0.151217, shoulder_lift_joint=-1.610439, elbow_joint=0.775573, wrist_1_joint=-0.735939, wrist_2_joint=-1.570760, wrist_3_joint=2.821707)}"/>

Commit message: Add native-contact PGI cup grasp simulation

File: urdf/pgi_140_80_macro.xacro (robot description, xacro)
@@ -31,5 +31,5 @@
   </xacro:macro>
   <xacro:macro name="pgi_140_80"
-               params="parent prefix camera_mount_xyz camera_mount_rpy use_gz_ros2_control:=false">
+               params="parent prefix camera_mount_xyz camera_mount_rpy use_gz_ros2_control:=false use_contact_physics:=false">
     <!-- The nominal and commandable travel remains 0.040 m per jaw. DART can
          latch a position-controlled prismatic joint after it is held exactly
@@ -40,4 +40,11 @@
     <xacro:if value="${use_gz_ros2_control}">
       <xacro:property name="pgi_physics_upper_limit" value="0.0405"/>
+    </xacro:if>
+    <!-- The standard logical model retains the full documented 140 N upper
+         limit.  The isolated Stage-5 contact variant starts at the documented
+         minimum selectable gripping force, 40 N per jaw. -->
+    <xacro:property name="pgi_effort_limit" value="140.0"/>
+    <xacro:if value="${use_contact_physics}">
+      <xacro:property name="pgi_effort_limit" value="40.0"/>
     </xacro:if>
     <!-- Placeholder camera interposer. Its final material, mass, and geometry
@@ -140,5 +147,5 @@
       <child link="${prefix}pgi_left_finger"/>
       <axis xyz="1 0 0"/>
-      <limit lower="0.0" upper="${pgi_physics_upper_limit}" effort="140.0" velocity="0.0364"/>
+      <limit lower="0.0" upper="${pgi_physics_upper_limit}" effort="${pgi_effort_limit}" velocity="0.0364"/>
       <!-- Provisional viscous damping for stable position control in Gazebo. -->
       <dynamics damping="2.0" friction="0.0"/>
@@ -163,8 +170,21 @@
       <child link="${prefix}pgi_right_finger"/>
       <axis xyz="-1 0 0"/>
-      <limit lower="0.0" upper="${pgi_physics_upper_limit}" effort="140.0" velocity="0.0364"/>
+      <limit lower="0.0" upper="${pgi_physics_upper_limit}" effort="${pgi_effort_limit}" velocity="0.0364"/>
       <dynamics damping="2.0" friction="0.0"/>
       <mimic joint="${prefix}pgi_left_finger_joint" multiplier="1.0" offset="0.0"/>
     </joint>
+    <!-- Stage-5-only provisional rubber/plastic contact parameters. They are
+         disabled in the saved logical baseline and require experimental
+         calibration before any result can be treated as predictive. -->
+    <xacro:if value="${use_contact_physics}">
+      <gazebo reference="${prefix}pgi_left_finger">
+        <mu1>1.5</mu1><mu2>1.5</mu2>
+        <kp>100000</kp><kd>50</kd><maxVel>0.02</maxVel><minDepth>0.0002</minDepth>
+      </gazebo>
+      <gazebo reference="${prefix}pgi_right_finger">
+        <mu1>1.5</mu1><mu2>1.5</mu2>
+        <kp>100000</kp><kd>50</kd><maxVel>0.02</maxVel><minDepth>0.0002</minDepth>
+      </gazebo>
+    </xacro:if>
     <!-- Logical grasp frame only. Cup and straw frames belong to the later
          attach/detach workflow and must not be hard-coded into this body. -->

File: urdf/ur_gz_feeding_markers.urdf.xacro (robot description, xacro)
@@ -32,4 +32,5 @@
   <xacro:arg name="use_pgi_gripper" default="false" />
   <xacro:arg name="use_pgi_sim_control" default="false" />
+  <xacro:arg name="pgi_contact_physics" default="false" />
   <xacro:arg name="pgi_logical_grasp_start" default="false" />
   <xacro:arg name="camera_mount_xyz" default="0 0.085 0.030" />
@@ -94,4 +95,5 @@
       camera_mount_rpy="$(arg camera_mount_rpy)"
       use_gz_ros2_control="$(arg use_pgi_sim_control)"
+      use_contact_physics="$(arg pgi_contact_physics)"
     />
   </xacro:if>

Commit message: Connect Grasp-Anything candidates to MoveIt simulation

File: urdf/pgi_140_80_macro.xacro (robot description, xacro)
@@ -41,11 +41,8 @@
       <xacro:property name="pgi_physics_upper_limit" value="0.0405"/>
     </xacro:if>
-    <!-- The standard logical model retains the full documented 140 N upper
-         limit.  The isolated Stage-5 contact variant starts at the documented
-         minimum selectable gripping force, 40 N per jaw. -->
+    <!-- Documented hardware upper limit. Individual simulation workflows use
+         separate controller YAML files to select 40 to 140 N without changing
+         this exact-model joint limit. -->
     <xacro:property name="pgi_effort_limit" value="140.0"/>
-    <xacro:if value="${use_contact_physics}">
-      <xacro:property name="pgi_effort_limit" value="40.0"/>
-    </xacro:if>
     <!-- Placeholder camera interposer. Its final material, mass, and geometry
          depend on the project adapter design. The 0.10 kg uniform-box inertia
